Commit message: Confirmed that robot can be controlled by both moveit and original joint-based interface

File: scara_robot_samples/urdf/common.xacro (robot description, xacro)
@@ -95,5 +95,5 @@
         <maxEffort>${max_effort}</maxEffort>              <!-- only taken into account if has_pid:=true [Nm] -->
         <xacro:unless value="${robot_namespace == ''}">
-          <robotNamespace>($robot_namespace)</robotNamespace>
+          <robotNamespace>$(arg robot_namespace)</robotNamespace>
         </xacro:unless>
       </plugin>

File: scara_robot_samples/urdf/scara_robot.urdf.xacro (robot description, xacro)
@@ -1,4 +1,5 @@
 <?xml version="1.0"?>
 <robot name="arm_robot" xmlns:xacro="http://www.ros.org/wiki/xacro">
+  <xacro:arg name="robot_namespace" default="/arm_robot"/>
   <xacro:include filename="$(find scara_robot_samples)/urdf/common.xacro"/>
   <link name="world"/>
@@ -207,5 +208,6 @@
       origin_x="0.0" origin_y="0.0" origin_z="-0.038115" axis_x="0" axis_y="1" axis_z="0">
     </xacro:armjoint>
-    <mimic joint="arm5r_joint" multiplier="-1" offset="0" />
+    <mimic joint="arm5r_joint" multiplier="-1" offset="0"
+	   robot_namespace="$(arg robot_namespace)"/>
   </joint>
   <xacro:mimic_joint_plugin_gazebo name_prefix="arm5l_joint"
@@ -235,7 +237,6 @@
   <gazebo>
     <plugin name="gazebo_ros_control" filename="libgazebo_ros_control.so">
-      <!-- <robotNamespace>/arm_robot</robotNamespace> -->
-      <robotNamespace>/</robotNamespace>
-      <!-- <robotSimType>gazebo_ros_control/DefaultRobotHWSim</robotSimType> -->
+      <robotNamespace>$(arg robot_namespace)</robotNamespace>
+      <robotSimType>gazebo_ros_control/DefaultRobotHWSim</robotSimType>
       <legacyModeNS>true</legacyModeNS>
     </plugin>
