Commit message: Add scara_robot_routines package

File: scara_robot_samples/urdf/scara_robot.urdf.xacro (robot description, xacro)
@@ -231,4 +231,10 @@
       </inertial>
     </link>
+    <link name="tip_link"/>
+    <joint name="tip_link_joint" type="fixed">
+      <parent link="arm4_link"/>
+      <child link="tip_link"/>
+      <origin rpy="0.0 ${pi/2} 0.0" xyz="0.0 0.0 -0.067"/>
+    </joint>
   <!--xacro:boxlink link_name="arm5l_link" mass="0.004" x="0" y="0" z="0" depth="0.023" width="0.001" height="0.023"/-->
   <gazebo reference="arm5l_link">
